File: kicad/eaterboard/eaterboard.kicad_pcb (KiCad board)
At the start: 2 copper layers, 3 parts, among them U1 W65C02SxP, U2 AT28C256-15PU, U3 W65C22NxP

Commit message: some more stuff
Parts:
- added C1: 0.1uF, Capacitor_Tantalum_SMD:CP_EIA-1608-08_AVX-J, F.Cu at (35.3, 72.0)
- added J1: Conn_02x20_Counter_Clockwise, Connector_PinSocket_2.54mm:PinSocket_2x20_P2.54mm_Vertical_SMD, F.Cu at (236.1, 95.6)
- added J2: Conn_01x02_Pin, Connector_PinSocket_2.54mm:PinSocket_1x02_P2.54mm_Vertical, F.Cu at (109.5, 163.5)
- added J4: Conn_02x10_Counter_Clockwise, Connector_PinSocket_2.54mm:PinSocket_2x10_P2.54mm_Vertical_SMD, F.Cu at (191.9, 157.0)
- added JP1: Jumper_3_Open, Jumper:SolderJumper-2_P1.3mm_Bridged2Bar_Pad1.0x1.5mm, F.Cu at (101.8, 166.5)
- added R1: 1k, Resistor_THT:R_Axial_DIN0204_L3.6mm_D1.6mm_P1.90mm_Vertical, F.Cu at (42.0, 74.5)
- added R2: 1k, Resistor_THT:R_Axial_DIN0204_L3.6mm_D1.6mm_P1.90mm_Vertical, F.Cu at (42.1, 69.0)
- added SW1: Reset, Button_Switch_THT:KSA_Tactile_SPST, F.Cu at (34.0, 54.7)
- added U4: 74HC00, Package_DIP:DIP-14_W7.62mm, F.Cu at (102.4, 62.3)
- added U5: CY62256-70PC, Package_DIP:DIP-28_W15.24mm, F.Cu at (118.5, 107.9)
- added Y1: ACO-1MHz, Oscillator:Oscillator_DIP-14, F.Cu at (41.9, 149.3)
- moved U3 92.5 mm to (168.0, 138.0), turned to 90 degrees
- moved U2 64.9 mm to (119.0, 81.4), turned to -90 degrees
- moved U1 24.9 mm to (60.0, 63.7)
Connections:
- U1 pad 34: unconnected-(U1-R/~{W}-Pad34) -> Net-(U1-R/~{W})
- U1 pad 37: unconnected-(U1-ϕ0-Pad37) -> CLOCK
- U1 pad 40: Net-(U1-~{RES}) -> RESET
- U3 pad 1: unconnected-(U3-VSS-Pad1) -> GND
- U3 pad 10: unconnected-(U3-PB0-Pad10) -> Net-(J4-Pin_20)
- U3 pad 11: unconnected-(U3-PB1-Pad11) -> Net-(J4-Pin_19)
- U3 pad 12: unconnected-(U3-PB2-Pad12) -> Net-(J4-Pin_18)
- U3 pad 13: unconnected-(U3-PB3-Pad13) -> Net-(J4-Pin_17)
- U3 pad 14: unconnected-(U3-PB4-Pad14) -> Net-(J4-Pin_16)
- U3 pad 15: unconnected-(U3-PB5-Pad15) -> Net-(J4-Pin_15)
- U3 pad 16: unconnected-(U3-PB6-Pad16) -> Net-(J4-Pin_14)
- U3 pad 17: unconnected-(U3-PB7-Pad17) -> Net-(J4-Pin_13)
- U3 pad 18: unconnected-(U3-CB1-Pad18) -> Net-(J4-Pin_12)
- U3 pad 19: unconnected-(U3-CB2-Pad19) -> Net-(J4-Pin_11)
- U3 pad 2: unconnected-(U3-PA0-Pad2) -> Net-(J4-Pin_1)
- U3 pad 20: unconnected-(U3-VCC-Pad20) -> +5V
- U3 pad 22: unconnected-(U3-R/~{W}-Pad22) -> Net-(U1-R/~{W})
- U3 pad 23: unconnected-(U3-~{CS2}-Pad23) -> Net-(U3-~{CS2})
- U3 pad 24: unconnected-(U3-CS1-Pad24) -> /A13
- U3 pad 25: unconnected-(U3-ϕ2-Pad25) -> CLOCK
- U3 pad 3: unconnected-(U3-PA1-Pad3) -> Net-(J4-Pin_2)
- U3 pad 34: unconnected-(U3-~{RES}-Pad34) -> RESET
- U3 pad 35: unconnected-(U3-RS3-Pad35) -> /A3
- U3 pad 36: unconnected-(U3-RS2-Pad36) -> /A2
- U3 pad 37: unconnected-(U3-RS1-Pad37) -> /A1
- U3 pad 38: unconnected-(U3-RS0-Pad38) -> /A0
- U3 pad 39: unconnected-(U3-CA2-Pad39) -> Net-(J4-Pin_10)
- U3 pad 4: unconnected-(U3-PA2-Pad4) -> Net-(J4-Pin_3)
- U3 pad 40: unconnected-(U3-CA1-Pad40) -> Net-(J4-Pin_9)
- U3 pad 5: unconnected-(U3-PA3-Pad5) -> Net-(J4-Pin_4)
- U3 pad 6: unconnected-(U3-PA4-Pad6) -> Net-(J4-Pin_5)
- U3 pad 7: unconnected-(U3-PA5-Pad7) -> Net-(J4-Pin_6)
- U3 pad 8: unconnected-(U3-PA6-Pad8) -> Net-(J4-Pin_7)
- U3 pad 9: unconnected-(U3-PA7-Pad9) -> Net-(J4-Pin_8)
Routing:
- net /D7: track 0.00 -> 22.0 mm
- net /D6: track 0.00 -> 19.9 mm
- net /D0: track 0.00 -> 19.3 mm
- net /D5: track 0.00 -> 18.1 mm
- net /D1: track 0.00 -> 18.0 mm
- net /D4: track 0.00 -> 16.3 mm
- net /D2: track 0.00 -> 15.4 mm
- net /D3: track 0.00 -> 13.9 mm
