File: kicad/eaterboard/eaterboard.kicad_sch (KiCad schematic)
At the start: 12 parts, among them J1 Conn_02x20_Counter_Clockwise, SW1 Reset, U1 W65C02SxP, U2 AT28C256-15PU, U3 W65C22NxP, U4 74HC00, U5 CY62256-70PC, Y1 ACO-1MHz

Commit message: some more stuff
Parts:
- added J2: External Clock Input, Connector_PinSocket_2.54mm:PinSocket_1x02_P2.54mm_Vertical, symbol Connector:Conn_01x02_Pin
- added J4: Conn_02x10_Counter_Clockwise, Connector_PinSocket_2.54mm:PinSocket_2x10_P2.54mm_Vertical_SMD, symbol Connector_Generic:Conn_02x10_Counter_Clockwise
- C1: footprint (none) -> Capacitor_Tantalum_SMD:CP_EIA-1608-08_AVX-J
- J1: footprint (none) -> Connector_PinSocket_2.54mm:PinSocket_2x20_P2.54mm_Vertical_SMD
- JP1: value Jumper_3_Open -> Clock Selector; footprint (none) -> Jumper:SolderJumper-2_P1.3mm_Bridged2Bar_Pad1.0x1.5mm
- R1, R2: footprint (none) -> Resistor_THT:R_Axial_DIN0204_L3.6mm_D1.6mm_P1.90mm_Vertical
- SW1: footprint (none) -> Button_Switch_THT:KSA_Tactile_SPST
- U2: footprint 28P6_ATM -> Package_DIP:DIP-28_W15.24mm
- U4: footprint (none) -> Package_DIP:DIP-14_W7.62mm
Connections:
- net CLOCK: now also J1.21 (Pin_21), U1.37 (ϕ0), U3.25 (ϕ2)
- net GND: now also J1.20 (Pin_20)
- net at JP1.3 (B): now also J2.1 (Pin_1)
- net RESET: now reaches C1.1, R2.2, SW1.2, U1.40 (~{RES})
- net RESET: now also U3.34 (~{RES})
- net at U3.10 (PB0): now also J4.20 (Pin_20)
- net at U3.11 (PB1): now also J4.19 (Pin_19)
- net at U3.12 (PB2): now also J4.18 (Pin_18)
- net at U3.13 (PB3): now also J4.17 (Pin_17)
- net at U3.14 (PB4): now also J4.16 (Pin_16)
- net at U3.15 (PB5): now also J4.15 (Pin_15)
- net at U3.16 (PB6): now also J4.14 (Pin_14)
- net at U3.17 (PB7): now also J4.13 (Pin_13)
- net at U3.18 (CB1): now also J4.12 (Pin_12)
- net at U3.19 (CB2): now also J4.11 (Pin_11)
- net at U3.2 (PA0): now also J4.1 (Pin_1)
- net at U3.3 (PA1): now also J4.2 (Pin_2)
- net at U3.39 (CA2): now also J4.10 (Pin_10)
- net at U3.4 (PA2): now also J4.3 (Pin_3)
- net at U3.40 (CA1): now also J4.9 (Pin_9)
- net at U3.5 (PA3): now also J4.4 (Pin_4)
- net at U3.6 (PA4): now also J4.5 (Pin_5)
- net at U3.7 (PA5): now also J4.6 (Pin_6)
- net at U3.8 (PA6): now also J4.7 (Pin_7)
- net at U3.9 (PA7): now also J4.8 (Pin_8)
- no-connect marks 11 -> 24
Other:
- title: (none) -> JAWN25
